Commit message: It all seems to be working

File: src/description/urdf/robot.urdf (robot description, URDF)
Before this commit: robot robot, 13 links, 12 joints
Links:
- removed link backhoe_bucket
- removed link bucket
- removed link imu
- removed link monoboom
- removed link monoboom_actuator_link
Joints:
- removed joint central_drive_to_monoboom
- removed joint frame_to_bucket
- removed joint frame_to_imu
- removed joint monoboom_actuator
- removed joint monoboom_to_backhoe_bucket
- joint zr300_dynamixel_to_zr300_mount: type revolute -> fixed

Commit message: Full driving simulation up and running

File: src/description/urdf/robot.urdf (robot description, URDF)
Before this commit: robot robot, 8 links, 7 joints
Links:
- removed link zr300_dynamixel
- removed link zr300_mount
- removed link zr300_mount_2
Joints:
- removed joint computer_box_to_zr300_dynamixel
- removed joint zr300_dynamixel_to_zr300_mount
- removed joint zr300_mount_to_zr300_mount_2

Commit message: Started on gazebo stuff

File: src/description/urdf/robot.urdf (robot description, URDF)
Before this commit: robot robot, 5 links, 4 joints
Links:
- link base_link: mass None -> 1; geometry visual box size=0.001 0.001 0.001
- link battery_box: mass None -> 1
- link central_drive: mass None -> 1
- link computer_box: mass None -> 1
- link frame: mass None -> 1; geometry collision box size=0.001 0.001 0.001; visual mesh filename=package://description/meshes/frame.stl

Commit message: finished_urdf

File: src/description/urdf/robot.urdf (robot description, URDF)
Before this commit: robot robot, 5 links, 4 joints
Links:
- added link backhoe_monoboom; visual mesh filename=package://description/meshes/backhoe_monoboom.stl
- added link bucket_backhoe; visual mesh filename=package://description/meshes/backhoe_bucket.stl
- added link gravel_bucket; visual mesh filename=package://description/meshes/gravel_bucket.stl
- added link left_flap; visual mesh filename=package://description/meshes/left_flap.stl
- added link right_flap; visual mesh filename=package://description/meshes/right_flap.stl
- link battery_box: geometry visual mesh filename=package://description/meshes/battery_box.stl
- link computer_box: geometry visual mesh filename=package://description/meshes/computer_box.stl
Joints:
- removed joint frame_to_battery_box
- removed joint frame_to_computer_box
- added joint battery_box_to_base: type fixed, parent base_link, child battery_box, origin xyz=0 0 0 rpy=0 0 0
- added joint bucket_to_monoboom: type revolute, parent backhoe_monoboom, child bucket_backhoe, origin xyz=0.55 0 0 rpy=0 0 3.14, axis 0 0 1, limit lower=0 upper=2.25 effort=1000.0 velocity=1
- added joint computer_box_to_base: type fixed, parent base_link, child computer_box, origin xyz=0 0 0 rpy=0 0 0
- added joint frame_to_gravel_bucket: type revolute, parent frame, child gravel_bucket, origin xyz=0 0 0 rpy=0 0 0, axis 0 -1 0, limit lower=0 upper=1.25 effort=1000.0 velocity=1.0
- added joint left_flap_joint: type revolute, parent frame, child left_flap, origin xyz=0.53 0.125 -0.2 rpy=1.57 0 -1.57, axis 0 0 1, limit lower=-1.55 upper=1.25 effort=1000.0 velocity=1.0
- added joint monoboom_to_frame: type revolute, parent frame, child backhoe_monoboom, origin xyz=0.98 0 -0.365 rpy=1.57 0 3.14, axis 0 0 -1, limit lower=-1 upper=0.85 effort=1000.0 velocity=1.0
- added joint right_flap_joint: type revolute, parent frame, child right_flap, origin xyz=0.53 -0.125 -0.2 rpy=1.57 0 -1.57, axis 0 0 -1, limit lower=-1.55 upper=1.25 effort=1000.0 velocity=1.0
- joint frame_to_central_drive: origin xyz=0.5291836 0.0 0.079375 rpy=0 0 0 -> xyz=0 0 0 rpy=0 0 0

Commit message: Fixed central drive components

File: src/description/urdf/robot.urdf (robot description, URDF)
Before this commit: robot robot, 10 links, 9 joints
Joints:
- joint bucket_to_monoboom: type revolute -> ${central_drive_joints_type}
- joint frame_to_gravel_bucket: type revolute -> ${central_drive_joints_type}
- joint left_flap_joint: type revolute -> ${central_drive_joints_type}
- joint monoboom_to_frame: origin xyz=0.98 0 -0.365 rpy=1.57 0 3.14 -> xyz=0.98 0 -0.365 rpy=1.57 ${monoboom_angle} 3.14; type revolute -> ${central_drive_joints_type}
- joint right_flap_joint: type revolute -> ${central_drive_joints_type}

Commit message: Fixed naming convention issue

File: src/description/urdf/robot.urdf (robot description, URDF)
Before this commit: robot robot, 10 links, 9 joints
Joints:
- removed joint bucket_to_monoboom
- removed joint monoboom_to_frame
- added joint frame_to_monoboom: type ${central_drive_joints_type}, parent frame, child backhoe_monoboom, origin xyz=0.98 0 -0.365 rpy=1.57 ${monoboom_angle} 3.14, axis 0 0 -1, limit lower=-1 upper=0.85 effort=1000.0 velocity=1.0
- added joint monoboom_to_bucket: type ${central_drive_joints_type}, parent backhoe_monoboom, child bucket_backhoe, origin xyz=0.55 0 0 rpy=0 0 3.14, axis 0 0 1, limit lower=0 upper=2.25 effort=1000.0 velocity=1

Commit message: Fixedish the urdf

File: src/description/urdf/robot.urdf (robot description, URDF)
Before this commit: robot robot, 10 links, 9 joints
Joints:
- removed joint battery_box_to_base
- removed joint computer_box_to_base
- added joint frame_to_battery_box: type fixed, parent frame, child battery_box, origin xyz=387.35e-3 0 -2.0796e-01 rpy=0 0 0
- added joint frame_to_computer_box: type fixed, parent frame, child computer_box, origin xyz=387.35e-3 0 -2.0796e-01 rpy=0 0 0
- joint base_link_to_frame: origin xyz=-387.35e-3 0 2.0796e-01 rpy=0 0 0 -> xyz=-0.5 0 0.65 rpy=0 0 0

Commit message: moved robot out of the ground a bit

File: src/description/urdf/robot.urdf (robot description, URDF)
Before this commit: robot robot, 10 links, 9 joints
Joints:
- joint base_link_to_frame: origin xyz=-387.35e-3 0 2.0796e-01 rpy=0 0 0 -> xyz=-387.35e-3 0 .5 rpy=0 0 0

Commit message: Fixed urdf conflicts

File: src/description/urdf/robot.urdf (robot description, URDF)
Before this commit: robot robot, 10 links, 9 joints
Joints:
- removed joint battery_box_to_base
- removed joint computer_box_to_base
- added joint frame_to_battery_box: type fixed, parent frame, child battery_box, origin xyz=387.35e-3 0 -2.0796e-01 rpy=0 0 0
- added joint frame_to_computer_box: type fixed, parent frame, child computer_box, origin xyz=387.35e-3 0 -2.0796e-01 rpy=0 0 0
- joint base_link_to_frame: origin xyz=-387.35e-3 0 .5 rpy=0 0 0 -> xyz=-0.5 0 0.65 rpy=0 0 0

Commit message: Updated urdf

File: src/description/urdf/robot.urdf (robot description, URDF)
Before this commit: robot robot, 10 links, 9 joints
Links:
- added link left_camera; visual mesh filename=package://description/meshes/nodey_camera.stl
- added link left_nodey_mount; visual mesh filename=package://description/meshes/left_nodey.stl
- added link right_camera; visual mesh filename=package://description/meshes/nodey_camera.stl
- added link right_nodey_mount; visual mesh filename=package://description/meshes/right_nodey.stl
- link computer_box: geometry visual mesh filename=package://description/meshes/battery_box.stl
Joints:
- added joint left_nodey_fixed: type fixed, parent frame, child left_nodey_mount, origin xyz=0 0 0 rpy=0 0 0
- added joint left_nodey_joint: type revolute, parent left_nodey_mount, child left_camera, origin xyz=-0.035 0.32 0.04 rpy=0 1.57 0, limit lower=-4 upper=1 effort=1000.0 velocity=1.0
- added joint right_nodey_fixed: type fixed, parent frame, child right_nodey_mount, origin xyz=0 0 0 rpy=0 0 0
- added joint right_nodey_joint: type revolute, parent right_nodey_mount, child right_camera, origin xyz=-0.035 -0.32 0.04 rpy=0 1.57 0, limit lower=-1 upper=4 effort=1000.0 velocity=1.0
- joint battery_box_to_base: parent base_link -> frame
- joint computer_box_to_base: parent base_link -> frame

Commit message: Updated urdf for current test config

File: src/description/urdf/robot.urdf (robot description, URDF)
Before this commit: robot robot, 14 links, 13 joints
Links:
- removed link left_nodey_mount
- removed link right_nodey_mount
- added link left_tracker_mount; visual mesh filename=package://description/meshes/left_tracker.stl
- added link right_tracker_mount; visual mesh filename=package://description/meshes/right_tracker.stl
- link left_camera: geometry visual mesh filename=package://description/meshes/tracker_camera.stl
- link right_camera: geometry visual mesh filename=package://description/meshes/tracker_camera.stl
Joints:
- removed joint left_nodey_fixed
- removed joint left_nodey_joint
- removed joint right_nodey_fixed
- removed joint right_nodey_joint
- added joint left_tracker_fixed: type fixed, parent frame, child left_tracker_mount, origin xyz=0 0 0 rpy=0 0 0
- added joint left_tracker_joint: type revolute, parent left_tracker_mount, child left_camera, origin xyz=-0.035 0.32 0.04 rpy=0 1.57 0, limit lower=-4 upper=1 effort=1000.0 velocity=1.0
- added joint right_tracker_fixed: type fixed, parent frame, child right_tracker_mount, origin xyz=0 0 0 rpy=0 0 0
- added joint right_tracker_joint: type revolute, parent right_tracker_mount, child right_camera, origin xyz=-0.035 -0.32 0.04 rpy=0 1.57 0, limit lower=-1 upper=4 effort=1000.0 velocity=1.0

Commit message: Tag pose estimates are working

File: src/description/urdf/robot.urdf (robot description, URDF)
Before this commit: robot robot, 14 links, 13 joints
Joints:
- joint right_tracker_joint: origin xyz=-0.035 -0.32 0.04 rpy=0 1.57 0 -> xyz=-0.035 -0.32 0.04 rpy=0 ${pi} 0

Commit message: Updated left tracker urdf

File: src/description/urdf/robot.urdf (robot description, URDF)
Before this commit: robot robot, 14 links, 13 joints
Joints:
- joint left_tracker_joint: origin xyz=-0.035 0.32 0.04 rpy=0 1.57 0 -> xyz=-0.035 0.32 0.04 rpy=${-pi/2} 0 0

Commit message: Added tag 0 and 1 to the urdf

File: src/description/urdf/robot.urdf (robot description, URDF)
Before this commit: robot robot, 14 links, 13 joints
Links:
- added link tag0
- added link tag1
Joints:
- added joint map_to_tag0: type fixed, parent map, child tag0, origin xyz=0 -0.5025 0.2563 rpy=${pi/2} 0 ${pi/2}
- added joint map_to_tag1: type fixed, parent map, child tag1, origin xyz=0 0.5025 0.2563 rpy=${pi/2} 0 ${pi/2}

Commit message: Finished pose estimation

File: src/description/urdf/robot.urdf (robot description, URDF)
Before this commit: robot robot, 16 links, 15 joints
Links:
- added link tag4
Joints:
- added joint map_to_tag4: type fixed, parent map, child tag4, origin xyz=0 -0.5025 0.2563 rpy=${pi/2} 0 ${pi/2}
- joint right_tracker_fixed: origin xyz=0 0 0 rpy=0 0 0 -> xyz=-0.035 -0.32 0.04 rpy=0 0 0
- joint right_tracker_joint: origin xyz=-0.035 -0.32 0.04 rpy=0 ${pi} 0 -> xyz=0 0 0 rpy=0 ${pi} 0

Commit message: Good to go

File: src/description/urdf/robot.urdf (robot description, URDF)
Before this commit: robot robot, 17 links, 16 joints
Links:
- added link right_camera_base
Joints:
- added joint right_tracker_joint_2: type floating, parent right_camera_base, child right_camera, origin xyz=0 0 0 rpy=0 0 0
- joint right_tracker_joint: child right_camera -> right_camera_base; origin xyz=0 0 0 rpy=0 ${pi} 0 -> xyz=0 0 0 rpy=${pi/2} ${pi} 0; type revolute -> fixed

Commit message: Made mods

File: src/description/urdf/robot.urdf (robot description, URDF)
Before this commit: robot robot, 18 links, 17 joints
Joints:
- joint right_tracker_joint_2: limit (none) -> lower=-4 upper=1 effort=1000.0 velocity=1.0; type floating -> revolute

Commit message: Started fixing visuals

File: src/description/urdf/robot.urdf (robot description, URDF)
Before this commit: robot robot, 18 links, 17 joints
Links:
- removed link tag0
- removed link tag1
- removed link tag4
Joints:
- removed joint map_to_tag0
- removed joint map_to_tag1
- removed joint map_to_tag4

Commit message: Monoboom is correctly mapped

File: src/description/urdf/robot.urdf (robot description, URDF)
Before this commit: robot robot, 15 links, 14 joints
Links:
- removed link central_drive
Joints:
- removed joint frame_to_central_drive
- joint frame_to_gravel_bucket: type ${central_drive_joints_type} -> ${central_drive_joint_type}
- joint frame_to_monoboom: type ${central_drive_joints_type} -> ${central_drive_joint_type}
- joint left_flap_joint: type ${central_drive_joints_type} -> ${central_drive_joint_type}
- joint monoboom_to_bucket: type ${central_drive_joints_type} -> ${central_drive_joint_type}
- joint right_flap_joint: type ${central_drive_joints_type} -> ${central_drive_joint_type}

Commit message: Finished backhoe angle

File: src/description/urdf/robot.urdf (robot description, URDF)
Before this commit: robot robot, 14 links, 13 joints
Joints:
- joint monoboom_to_bucket: origin xyz=0.55 0 0 rpy=0 0 3.14 -> xyz=0.55 0 0 rpy=0 0 ${20*pi/180}

Commit message: Added left camera to urdf

File: src/description/urdf/robot.urdf (robot description, URDF)
Before this commit: robot robot, 15 links, 14 joints
Links:
- removed link left_camera
- removed link left_tracker_mount
- removed link right_camera
- removed link right_camera_base
- removed link right_tracker_mount
Joints:
- removed joint left_tracker_fixed
- removed joint left_tracker_joint
- removed joint right_tracker_fixed
- removed joint right_tracker_joint
- removed joint right_tracker_joint_2
- joint right_flap_joint: origin xyz=0.53 -0.125 -0.2 rpy=1.57 0 -1.57 -> xyz=0.53 -0.125 -0.2 rpy=${pi/2} 0 -${pi/2}
