Commit message: Integrated localization

File: src/description/urdf/arena.urdf (robot description, URDF)
Before this commit: robot arena, 1 links, 0 joints
Links:
- added link hopper
- added link tag1
- added link tag1_pose
Joints:
- added joint hopper_to_tag1_position: type fixed, parent hopper, child tag1_pose, origin xyz=0.2159 -0.7234 0.2563 rpy=0 0 1.1310
- added joint map_to_hopper: type fixed, parent map, child hopper, origin xyz=0.48 1.075 0 rpy=0 0 0
- added joint tag1_pose_to_tag1: type fixed, parent tag1_pose, child tag1, origin xyz=0 0 0 rpy=${pi/2} 0 ${pi/2}

File: src/description/urdf/robot.urdf (robot description, URDF)
Before this commit: robot robot, 14 links, 13 joints
Links:
- added link central_drive
Joints:
- added joint frame_to_central_drive: type ${central_drive_joint_type}, parent frame, child central_drive, origin xyz=0 0 0 rpy=0 0 0, axis 0 1 0, limit lower=-1e9 upper=1e9 effort=1000.0 velocity=1000.0

Commit message: Removed extra software and added additional apriltags

File: src/description/urdf/arena.urdf (robot description, URDF)
Before this commit: robot arena, 4 links, 3 joints
Links:
- removed link tag1
- removed link tag1_pose
Joints:
- removed joint hopper_to_tag1_position
- removed joint tag1_pose_to_tag1
